Commit message: final description

File: jinpao_description/robot/jinpao.urdf (robot description, URDF)
Before this commit: robot jinpao, 8 links, 7 joints
Links:
- removed link camera_link
- removed link camera_optical
- removed link lidar_link
Joints:
- removed joint camera_joint
- removed joint camera_optical_mount
- removed joint lidar_mount

File: jinpao_description/robot/visual/castor.xacro (robot description, xacro)
@@ -44,11 +44,11 @@
     <xacro:castor_graphics
       name="right_front"
-      translation_x="${-CASTOR_SEPARATION_X/2}"
-      translation_y="${CASTOR_SEPARATION_Y/2}"
+      translation_x="${CASTOR_SEPARATION_X/2}"
+      translation_y="${-CASTOR_SEPARATION_Y/2}"
     />
     <xacro:castor_graphics
       name="left_rear"
-      translation_x="${CASTOR_SEPARATION_X/2}"
-      translation_y="${-CASTOR_SEPARATION_Y/2}"
+      translation_x="${-CASTOR_SEPARATION_X/2}"
+      translation_y="${CASTOR_SEPARATION_Y/2}"
     />
     <xacro:castor_graphics

File: jinpao_description/robot/visual/jinpao_rviz.xacro (robot description, xacro)
@@ -8,7 +8,4 @@
         <xacro:include filename="${visual_path}/base.xacro"/>
         <xacro:base_graphics package="${package}" mesh_path="${BASE_MESH_PATH}"/>
-        <!-- Add wheels -->
-        <xacro:include filename="${visual_path}/wheel.xacro"/>
-        <xacro:wheel_set_graphics/>
         <!-- Add castor -->
         <xacro:include filename="${visual_path}/castor.xacro"/>

File: jinpao_description/robot/visual/properties.xacro (robot description, xacro)
@@ -25,15 +25,3 @@
   <xacro:property name="CASTOR_SEPARATION_Y" value="${mp['castor_separation_y']}"/>
   <xacro:property name="CASTOR_COLOR" value="${mp['castor_color']}"/>
-  <!-- Pole Contact Properties-->
-  <xacro:property name="POLE_RADIUS" value="${mp['pole_radius']}"/>
-  <xacro:property name="POLE_HEIGHT" value="${mp['pole_height']}"/>
-  <xacro:property name="POLE_SEPARATION_X" value="${mp['pole_separation_x']}"/>
-  <xacro:property name="POLE_SEPARATION_Y" value="${mp['pole_separation_y']}"/>
-  <!-- LIDAR Visual Properties -->
-  <xacro:property name="LIDAR_RADIUS" value="${mp['lidar_radius']}"/>
-  <xacro:property name="LIDAR_THICKNESS" value="${mp['lidar_thickness']}"/>
-  <xacro:property name="LIDAR_OFFSET" value="${mp['lidar_offset']}"/>
-  <!-- CAMERA Visual Properties -->
-  <xacro:property name="CAMERA_OFFSET" value="${mp['camera_offset']}"/>
-  <xacro:property name="CAMERA_HEIGHT" value="${mp['camera_height']}"/>
 </robot>

File: jinpao_description/robot/visual/sensor.xacro (robot description, xacro)
@@ -3,35 +3,4 @@
   <!-- Contents-->
   <xacro:macro name="sensor_link" params="">
-    <link name="lidar_link">
-      <visual>
-        <geometry>
-          <cylinder radius="${LIDAR_RADIUS}" length="${LIDAR_THICKNESS}"/>
-        </geometry>
-      </visual>
-    </link>
-    <joint name="lidar_mount" type="fixed">
-      <origin xyz="${LIDAR_OFFSET} 0.0 ${(BASE_HEIGHT+LIDAR_THICKNESS)/2}"/>
-      <parent link="base_link"/>
-      <child link="lidar_link"/>
-    </joint>
-    <link name="camera_link">
-      <visual>
-          <origin xyz="0 0 0" rpy="0 0 0" />
-          <geometry>
-              <box size="0.025 0.09 0.025"/>
-          </geometry>
-      </visual>
-    </link>
-    <link name="camera_optical"/>
-    <joint name="camera_joint" type="fixed">
-        <parent link="base_link" />
-        <child link="camera_link" />
-        <origin xyz="${CAMERA_OFFSET} 0 ${CAMERA_HEIGHT}" />
-    </joint>
-    <joint name="camera_optical_mount" type="fixed">
-        <parent link="camera_link" />
-        <child link="camera_optical" />
-        <origin xyz="0 0 0" rpy="${-PI/2} 0 ${-PI/2}" />
-    </joint>
     <link name="imu_link"/>
     <joint name="imu_mount" type="fixed">
